Commit message: Added autorepeat parameter to joy node in map_joystick.launch

File: ros_packages/fetch_description/robots/fetch.urdf (robot description, URDF)
Before this commit: robot fetch, 26 links, 25 joints
Joints:
- joint l_wheel_joint: origin xyz=0.0012914 0.18738 0.055325 rpy=-6.123E-17 0 0 -> xyz=0.0012914 0.18738 0.059125 rpy=-6.123E-17 0 0
- joint r_wheel_joint: origin xyz=0.0012914 -0.18738 0.055325 rpy=-6.123E-17 0 0 -> xyz=0.0012914 -0.18738 0.059125 rpy=-6.123E-17 0 0

File: ros_packages/fetch_gazebo/fetch_gazebo/robots/fetch.gazebo.xacro (robot description, xacro)
@@ -3,8 +3,8 @@
   <!-- Base is modeled as a big tub sitting on floor, with two wheels -->
   <gazebo reference="base_link">
-    <kp>100000000.0</kp>
-    <kd>10.0</kd>
-    <mu1>0.1</mu1>
-    <mu2>0.1</mu2>
+    <kp>10000000.0</kp>
+    <kd>1000.0</kd>
+    <mu1>0.0</mu1>
+    <mu2>0.0</mu2>
     <fdir1>1 0 0</fdir1>
     <maxVel>10.0</maxVel>
@@ -12,20 +12,20 @@
   </gazebo>
   <gazebo reference="r_wheel_link">
-    <kp>100000.0</kp>
+    <kp>100000000.0</kp>
     <kd>100.0</kd>
-    <mu1>1</mu1>
-    <mu2>1</mu2>
-    <!-- <fdir1>1 0 0</fdir1> -->
-    <maxVel>1.5</maxVel>
+    <mu1>10.0</mu1>
+    <mu2>10.0</mu2>
+    <fdir1>0 1 0</fdir1>
+    <maxVel>10.0</maxVel>
     <minDepth>0.003</minDepth>
     <material>Gazebo/Black</material>
   </gazebo>
   <gazebo reference="l_wheel_link">
-    <kp>100000.0</kp>
+    <kp>100000000.0</kp>
     <kd>100.0</kd>
-    <mu1>1</mu1>
-    <mu2>1</mu2>
-    <!-- <fdir1>1 0 0</fdir1> -->
-    <maxVel>1.5</maxVel>
+    <mu1>10.0</mu1>
+    <mu2>10.0</mu2>
+    <fdir1>0 1 0</fdir1>
+    <maxVel>10.0</maxVel>
     <minDepth>0.003</minDepth>
     <material>Gazebo/Black</material>
